File: Chevron_signal.kicad_pcb (KiCad board)
At the start: 2 copper layers, 960 x 960 mm, 0 parts

Commit message: cv28 v1.0
Parts:
- added D1: LED_CV28, CV28D-FCC:LED_CV28, F.Cu at (285.4, 1006.9)
- added D10: LED_CV28, CV28D-FCC:LED_CV28, F.Cu at (427.1, 1008.2)
- added D11: LED_CV28, CV28D-FCC:LED_CV28, F.Cu at (442.6, 1008.4)
- added D12: LED_CV28, CV28D-FCC:LED_CV28, F.Cu at (459.1, 1008.2)
- added D13: LED_CV28, CV28D-FCC:LED_CV28, F.Cu at (479.1, 1007.7)
- added D14: LED_CV28, CV28D-FCC:LED_CV28, F.Cu at (498.1, 1007.9)
- added D15: LED_CV28, CV28D-FCC:LED_CV28, F.Cu at (516.5, 1008.5)
- added D16: LED_CV28, CV28D-FCC:LED_CV28, F.Cu at (533.1, 1007.7)
- added D17: LED_CV28, CV28D-FCC:LED_CV28, F.Cu at (550.1, 1008.1)
- added D18: LED_CV28, CV28D-FCC:LED_CV28, F.Cu at (565.4, 1007.6)
- added D19: LED_CV28, CV28D-FCC:LED_CV28, F.Cu at (580.6, 1007.7)
- added D2: LED_CV28, CV28D-FCC:LED_CV28, F.Cu at (299.5, 1006.8)
- added D20: LED_CV28, CV28D-FCC:LED_CV28, F.Cu at (595.5, 1008.0)
- added D21: LED_CV28, CV28D-FCC:LED_CV28, F.Cu at (419.5, 1082.1)
- added D22: LED_CV28, CV28D-FCC:LED_CV28, F.Cu at (418.1, 1090.7)
- added D23: LED_CV28, CV28D-FCC:LED_CV28, F.Cu at (418.1, 1094.3)
- added D24: LED_CV28, CV28D-FCC:LED_CV28, F.Cu at (418.1, 1098.0)
- added D3: LED_CV28, CV28D-FCC:LED_CV28, F.Cu at (313.1, 1007.0)
- added D4: LED_CV28, CV28D-FCC:LED_CV28, F.Cu at (326.6, 1007.7)
- added D5: LED_CV28, CV28D-FCC:LED_CV28, F.Cu at (342.0, 1007.5)
- added D6: LED_CV28, CV28D-FCC:LED_CV28, F.Cu at (357.5, 1007.0)
- added D7: LED_CV28, CV28D-FCC:LED_CV28, F.Cu at (373.6, 1007.2)
- added D8: LED_CV28, CV28D-FCC:LED_CV28, F.Cu at (391.6, 1007.7)
- added D9: LED_CV28, CV28D-FCC:LED_CV28, F.Cu at (409.6, 1008.2)

Commit message: cv28 v1.1
Parts:
- added D100: LED_CV28, CV28D-FCC:LED_CV28, F.Cu at (364.5, 290.5)
- added D101: LED_CV28, CV28D-FCC:LED_CV28, F.Cu at (371.8, 300.4)
- added D102: LED_CV28, CV28D-FCC:LED_CV28, F.Cu at (379.0, 310.4)
- added D103: LED_CV28, CV28D-FCC:LED_CV28, F.Cu at (386.3, 320.4)
- added D104: LED_CV28, CV28D-FCC:LED_CV28, F.Cu at (393.5, 330.4)
- added D105: LED_CV28, CV28D-FCC:LED_CV28, F.Cu at (400.8, 340.4)
- added D106: LED_CV28, CV28D-FCC:LED_CV28, F.Cu at (408.0, 350.4)
- added D107: LED_CV28, CV28D-FCC:LED_CV28, F.Cu at (415.3, 360.4)
- added D108: LED_CV28, CV28D-FCC:LED_CV28, F.Cu at (422.6, 370.3)
- added D109: LED_CV28, CV28D-FCC:LED_CV28, F.Cu at (429.8, 380.3)
- added D110: LED_CV28, CV28D-FCC:LED_CV28, F.Cu at (437.1, 390.3)
- added D111: LED_CV28, CV28D-FCC:LED_CV28, F.Cu at (444.3, 400.3)
- added D112: LED_CV28, CV28D-FCC:LED_CV28, F.Cu at (451.6, 410.3)
- added D113: LED_CV28, CV28D-FCC:LED_CV28, F.Cu at (458.8, 420.2)
- added D114: LED_CV28, CV28D-FCC:LED_CV28, F.Cu at (466.1, 430.2)
- added D115: LED_CV28, CV28D-FCC:LED_CV28, F.Cu at (473.3, 440.2)
- added D116: LED_CV28, CV28D-FCC:LED_CV28, F.Cu at (480.6, 450.2)
- added D117: LED_CV28, CV28D-FCC:LED_CV28, F.Cu at (487.8, 460.2)
- added D118: LED_CV28, CV28D-FCC:LED_CV28, F.Cu at (495.1, 470.2)
- added D119: LED_CV28, CV28D-FCC:LED_CV28, F.Cu at (502.4, 480.1)
- added D120: LED_CV28, CV28D-FCC:LED_CV28, F.Cu at (488.2, 700.0)
- added D121: LED_CV28, CV28D-FCC:LED_CV28, F.Cu at (480.9, 710.0)
- added D122: LED_CV28, CV28D-FCC:LED_CV28, F.Cu at (473.7, 720.0)
- added D123: LED_CV28, CV28D-FCC:LED_CV28, F.Cu at (466.4, 730.0)
- added D124: LED_CV28, CV28D-FCC:LED_CV28, F.Cu at (459.1, 740.0)
- added D125: LED_CV28, CV28D-FCC:LED_CV28, F.Cu at (451.9, 750.0)
- added D126: LED_CV28, CV28D-FCC:LED_CV28, F.Cu at (444.6, 760.0)
- added D127: LED_CV28, CV28D-FCC:LED_CV28, F.Cu at (437.3, 770.0)
- added D128: LED_CV28, CV28D-FCC:LED_CV28, F.Cu at (430.0, 780.0)
- added D129: LED_CV28, CV28D-FCC:LED_CV28, F.Cu at (422.8, 790.0)
- added D130: LED_CV28, CV28D-FCC:LED_CV28, F.Cu at (415.5, 800.1)
- added D131: LED_CV28, CV28D-FCC:LED_CV28, F.Cu at (408.2, 810.1)
- added D132: LED_CV28, CV28D-FCC:LED_CV28, F.Cu at (400.9, 820.1)
- added D133: LED_CV28, CV28D-FCC:LED_CV28, F.Cu at (393.6, 830.1)
- added D134: LED_CV28, CV28D-FCC:LED_CV28, F.Cu at (386.4, 840.1)
- added D135: LED_CV28, CV28D-FCC:LED_CV28, F.Cu at (379.1, 850.1)
- added D136: LED_CV28, CV28D-FCC:LED_CV28, F.Cu at (371.8, 860.1)
- added D137: LED_CV28, CV28D-FCC:LED_CV28, F.Cu at (364.6, 870.1)
- added D138: LED_CV28, CV28D-FCC:LED_CV28, F.Cu at (357.3, 880.1)
- added D139: LED_CV28, CV28D-FCC:LED_CV28, F.Cu at (350.0, 890.1)
- added D140: LED_CV28, CV28D-FCC:LED_CV28, F.Cu at (342.7, 900.1)
- added D141: LED_CV28, CV28D-FCC:LED_CV28, F.Cu at (335.4, 910.1)
- added D142: LED_CV28, CV28D-FCC:LED_CV28, F.Cu at (328.2, 920.1)
- added D143: LED_CV28, CV28D-FCC:LED_CV28, F.Cu at (320.9, 930.1)
- added D144: LED_CV28, CV28D-FCC:LED_CV28, F.Cu at (313.6, 940.1)
- added D25: LED_CV28, CV28D-FCC:LED_CV28, F.Cu at (700.6, 891.5)
- added D26: LED_CV28, CV28D-FCC:LED_CV28, F.Cu at (707.8, 881.5)
- added D27: LED_CV28, CV28D-FCC:LED_CV28, F.Cu at (715.8, 871.6)
- added D28: LED_CV28, CV28D-FCC:LED_CV28, F.Cu at (722.8, 861.6)
- added D29: LED_CV28, CV28D-FCC:LED_CV28, F.Cu at (730.6, 851.9)
- added D30: LED_CV28, CV28D-FCC:LED_CV28, F.Cu at (736.8, 841.6)
- added D31: LED_CV28, CV28D-FCC:LED_CV28, F.Cu at (743.8, 831.6)
- added D32: LED_CV28, CV28D-FCC:LED_CV28, F.Cu at (751.2, 821.6)
- added D33: LED_CV28, CV28D-FCC:LED_CV28, F.Cu at (759.8, 811.4)
- added D34: LED_CV28, CV28D-FCC:LED_CV28, F.Cu at (766.8, 801.9)
- added D35: LED_CV28, CV28D-FCC:LED_CV28, F.Cu at (772.8, 791.6)
- added D36: LED_CV28, CV28D-FCC:LED_CV28, F.Cu at (780.9, 781.9)
- added D37: LED_CV28, CV28D-FCC:LED_CV28, F.Cu at (788.2, 771.6)
- added D38: LED_CV28, CV28D-FCC:LED_CV28, F.Cu at (795.8, 761.6)
- added D39: LED_CV28, CV28D-FCC:LED_CV28, F.Cu at (803.8, 751.6)
- added D40: LED_CV28, CV28D-FCC:LED_CV28, F.Cu at (810.8, 741.6)
- added D41: LED_CV28, CV28D-FCC:LED_CV28, F.Cu at (817.4, 731.9)
- added D42: LED_CV28, CV28D-FCC:LED_CV28, F.Cu at (825.9, 721.9)
- added D43: LED_CV28, CV28D-FCC:LED_CV28, F.Cu at (832.9, 711.9)
- added D44: LED_CV28, CV28D-FCC:LED_CV28, F.Cu at (839.9, 701.9)
- added D45: LED_CV28, CV28D-FCC:LED_CV28, F.Cu at (846.9, 691.9)
- added D46: LED_CV28, CV28D-FCC:LED_CV28, F.Cu at (854.9, 681.9)
- added D47: LED_CV28, CV28D-FCC:LED_CV28, F.Cu at (861.2, 671.6)
- added D48: LED_CV28, CV28D-FCC:LED_CV28, F.Cu at (864.7, 500.2)
- added D49: LED_CV28, CV28D-FCC:LED_CV28, F.Cu at (857.7, 490.2)
- added D50: LED_CV28, CV28D-FCC:LED_CV28, F.Cu at (850.8, 480.2)
- added D51: LED_CV28, CV28D-FCC:LED_CV28, F.Cu at (843.8, 470.3)
- added D52: LED_CV28, CV28D-FCC:LED_CV28, F.Cu at (836.8, 460.3)
- added D53: LED_CV28, CV28D-FCC:LED_CV28, F.Cu at (829.9, 450.3)
- added D54: LED_CV28, CV28D-FCC:LED_CV28, F.Cu at (822.9, 440.3)
- added D55: LED_CV28, CV28D-FCC:LED_CV28, F.Cu at (815.9, 430.4)
- added D56: LED_CV28, CV28D-FCC:LED_CV28, F.Cu at (809.0, 420.4)
- added D57: LED_CV28, CV28D-FCC:LED_CV28, F.Cu at (802.0, 410.4)
- added D58: LED_CV28, CV28D-FCC:LED_CV28, F.Cu at (795.0, 400.4)
- added D59: LED_CV28, CV28D-FCC:LED_CV28, F.Cu at (788.1, 390.5)
- added D60: LED_CV28, CV28D-FCC:LED_CV28, F.Cu at (781.1, 380.5)
- added D61: LED_CV28, CV28D-FCC:LED_CV28, F.Cu at (774.1, 370.5)
- added D62: LED_CV28, CV28D-FCC:LED_CV28, F.Cu at (767.2, 360.5)
- added D63: LED_CV28, CV28D-FCC:LED_CV28, F.Cu at (760.2, 350.5)
- added D64: LED_CV28, CV28D-FCC:LED_CV28, F.Cu at (753.3, 340.6)
- added D65: LED_CV28, CV28D-FCC:LED_CV28, F.Cu at (746.3, 330.6)
- added D66: LED_CV28, CV28D-FCC:LED_CV28, F.Cu at (739.3, 320.6)
- added D67: LED_CV28, CV28D-FCC:LED_CV28, F.Cu at (732.4, 310.6)
- added D68: LED_CV28, CV28D-FCC:LED_CV28, F.Cu at (725.4, 300.7)
- added D69: LED_CV28, CV28D-FCC:LED_CV28, F.Cu at (718.4, 290.7)
- added D70: LED_CV28, CV28D-FCC:LED_CV28, F.Cu at (711.5, 280.7)
- added D71: LED_CV28, CV28D-FCC:LED_CV28, F.Cu at (704.5, 270.7)
- added D72: LED_CV28, CV28D-FCC:LED_CV28, F.Cu at (697.5, 260.8)
- added D73: LED_CV28, CV28D-FCC:LED_CV28, F.Cu at (690.6, 250.8)
- added D74: LED_CV28, CV28D-FCC:LED_CV28, F.Cu at (683.6, 240.8)
- added D75: LED_CV28, CV28D-FCC:LED_CV28, F.Cu at (612.5, 160.6)
- added D76: LED_CV28, CV28D-FCC:LED_CV28, F.Cu at (594.9, 160.0)
- added D77: LED_CV28, CV28D-FCC:LED_CV28, F.Cu at (577.4, 160.0)
- added D78: LED_CV28, CV28D-FCC:LED_CV28, F.Cu at (559.8, 159.9)
- added D79: LED_CV28, CV28D-FCC:LED_CV28, F.Cu at (542.2, 160.1)
- added D80: LED_CV28, CV28D-FCC:LED_CV28, F.Cu at (524.7, 160.1)
- added D81: LED_CV28, CV28D-FCC:LED_CV28, F.Cu at (507.1, 160.1)
- added D82: LED_CV28, CV28D-FCC:LED_CV28, F.Cu at (489.5, 160.2)
- added D83: LED_CV28, CV28D-FCC:LED_CV28, F.Cu at (472.0, 160.5)
- added D84: LED_CV28, CV28D-FCC:LED_CV28, F.Cu at (454.4, 160.4)
- added D85: LED_CV28, CV28D-FCC:LED_CV28, F.Cu at (436.8, 160.4)
- added D86: LED_CV28, CV28D-FCC:LED_CV28, F.Cu at (419.3, 159.9)
- added D87: LED_CV28, CV28D-FCC:LED_CV28, F.Cu at (401.7, 160.2)
- added D88: LED_CV28, CV28D-FCC:LED_CV28, F.Cu at (384.1, 160.2)
- added D89: LED_CV28, CV28D-FCC:LED_CV28, F.Cu at (366.6, 159.9)
- added D90: LED_CV28, CV28D-FCC:LED_CV28, F.Cu at (349.0, 160.3)
- added D91: LED_CV28, CV28D-FCC:LED_CV28, F.Cu at (331.4, 160.3)
- added D92: LED_CV28, CV28D-FCC:LED_CV28, F.Cu at (313.9, 160.4)
- added D93: LED_CV28, CV28D-FCC:LED_CV28, F.Cu at (296.3, 160.5)
- added D94: LED_CV28, CV28D-FCC:LED_CV28, F.Cu at (278.7, 160.5)
- added D95: LED_CV28, CV28D-FCC:LED_CV28, F.Cu at (328.2, 240.6)
- added D96: LED_CV28, CV28D-FCC:LED_CV28, F.Cu at (335.5, 250.5)
- added D97: LED_CV28, CV28D-FCC:LED_CV28, F.Cu at (342.8, 260.5)
- added D98: LED_CV28, CV28D-FCC:LED_CV28, F.Cu at (350.0, 270.5)
- added D99: LED_CV28, CV28D-FCC:LED_CV28, F.Cu at (357.3, 280.5)
- added P1: 282837-2, 282837-2:TE_282837-2, F.Cu at (964.5, 899.5)
- added R1: R_Small, Resistor_THT:R_Axial_DIN0617_L17.0mm_D6.0mm_P20.32mm_Horizontal, F.Cu at (1007.2, 981.5)
- added R2: R_Small, Resistor_THT:R_Axial_DIN0617_L17.0mm_D6.0mm_P20.32mm_Horizontal, F.Cu at (1007.2, 974.0)
- added R3: R_Small, Resistor_THT:R_Axial_DIN0617_L17.0mm_D6.0mm_P20.32mm_Horizontal, F.Cu at (1007.2, 966.5)
- added R4: R_Small, Resistor_THT:R_Axial_DIN0617_L17.0mm_D6.0mm_P20.32mm_Horizontal, F.Cu at (960.6, 875.8)
- added R5: R_Small, Resistor_THT:R_Axial_DIN0617_L17.0mm_D6.0mm_P20.32mm_Horizontal, F.Cu at (960.6, 883.3)
- added R6: R_Small, Resistor_THT:R_Axial_DIN0617_L17.0mm_D6.0mm_P20.32mm_Horizontal, F.Cu at (960.6, 890.9)
- moved D24 337.7 mm to (693.1, 902.0)
- moved D23 323.8 mm to (685.6, 911.9)
- moved D22 309.8 mm to (677.6, 921.5)
- moved D21 292.8 mm to (670.6, 931.6)
- moved D7 22.3 mm to (395.1, 1001.4)
- moved D6 22.0 mm to (378.8, 1001.4)
- moved D5 21.4 mm to (362.5, 1001.4)
- moved D8 20.8 mm to (411.5, 1001.4)
- moved D4 20.6 mm to (346.2, 1001.4)
- moved D9 19.4 mm to (427.8, 1001.4)
- moved D11 19.1 mm to (460.4, 1001.4)
- moved D12 18.9 mm to (476.7, 1001.4)
- moved D10 18.3 mm to (444.1, 1001.4)
- moved D3 17.7 mm to (329.9, 1001.4)
- moved D13 15.3 mm to (493.1, 1001.4)
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Connections:
- D1 pad A1: unconnected-(D1-PadA1) -> Net-(D1-PadA1)
- D1 pad A2: unconnected-(D1-PadA2) -> Net-(D1-PadA2)
- D1 pad A3: unconnected-(D1-PadA3) -> Net-(D1-PadA3)
- D1 pad C2: unconnected-(D1-PadC2) -> Net-(D1-PadC2)
- D1 pad C3: unconnected-(D1-PadC3) -> Net-(D1-PadC3)
- D10 pad C1: Net-(D10-PadC1) -> unconnected-(D10-PadC1)
- D11 pad A1: Net-(D10-PadC1) -> unconnected-(D11-PadA1)
- D11 pad C1: Net-(D11-PadC1) -> unconnected-(D11-PadC1)
- D12 pad A1: Net-(D11-PadC1) -> unconnected-(D12-PadA1)
- D13 pad C1: Net-(D13-PadC1) -> unconnected-(D13-PadC1)
- D14 pad A1: Net-(D13-PadC1) -> unconnected-(D14-PadA1)
- D14 pad C1: Net-(D14-PadC1) -> unconnected-(D14-PadC1)
- D15 pad A1: Net-(D14-PadC1) -> unconnected-(D15-PadA1)
- D16 pad C1: Net-(D16-PadC1) -> unconnected-(D16-PadC1)
- D17 pad A1: Net-(D16-PadC1) -> unconnected-(D17-PadA1)
- D17 pad C1: Net-(D17-PadC1) -> unconnected-(D17-PadC1)
- D18 pad A1: Net-(D17-PadC1) -> unconnected-(D18-PadA1)
- D19 pad C1: Net-(D19-PadC1) -> unconnected-(D19-PadC1)
- D2 pad A2: unconnected-(D2-PadA2) -> Net-(D1-PadC2)
- D2 pad A3: unconnected-(D2-PadA3) -> Net-(D1-PadC3)
- D2 pad C2: unconnected-(D2-PadC2) -> Net-(D2-PadC2)
- D2 pad C3: unconnected-(D2-PadC3) -> Net-(D2-PadC3)
- D20 pad A1: Net-(D19-PadC1) -> unconnected-(D20-PadA1)
- D20 pad C1: Net-(D20-PadC1) -> unconnected-(D20-PadC1)
- D21 pad A1: Net-(D20-PadC1) -> unconnected-(D21-PadA1)
- D22 pad C1: Net-(D22-PadC1) -> unconnected-(D22-PadC1)
- D23 pad A1: Net-(D22-PadC1) -> unconnected-(D23-PadA1)
- D23 pad C1: Net-(D23-PadC1) -> unconnected-(D23-PadC1)
- D24 pad A1: Net-(D23-PadC1) -> unconnected-(D24-PadA1)
- D3 pad A2: unconnected-(D3-PadA2) -> Net-(D2-PadC2)
- D3 pad A3: unconnected-(D3-PadA3) -> Net-(D2-PadC3)
- D3 pad C1: unconnected-(D3-PadC1) -> Net-(D3-PadC1)
- D3 pad C2: unconnected-(D3-PadC2) -> Net-(D3-PadC2)
- D3 pad C3: unconnected-(D3-PadC3) -> GND
- D4 pad A1: unconnected-(D4-PadA1) -> Net-(D3-PadC1)
- D4 pad A2: unconnected-(D4-PadA2) -> Net-(D3-PadC2)
- D4 pad A3: unconnected-(D4-PadA3) -> Net-(D4-PadA3)
- D4 pad C1: Net-(D4-PadC1) -> GND
- D4 pad C2: unconnected-(D4-PadC2) -> GND
- D4 pad C3: unconnected-(D4-PadC3) -> Net-(D4-PadC3)
- D5 pad A1: Net-(D4-PadC1) -> Net-(D5-PadA1)
- D5 pad A2: unconnected-(D5-PadA2) -> Net-(D5-PadA2)
- D5 pad A3: unconnected-(D5-PadA3) -> Net-(D4-PadC3)
- D5 pad C2: unconnected-(D5-PadC2) -> Net-(D5-PadC2)
- D5 pad C3: unconnected-(D5-PadC3) -> Net-(D5-PadC3)
- D6 pad A2: unconnected-(D6-PadA2) -> Net-(D5-PadC2)
- D6 pad A3: unconnected-(D6-PadA3) -> Net-(D5-PadC3)
- D6 pad C1: unconnected-(D6-PadC1) -> Net-(D6-PadC1)
- D6 pad C2: unconnected-(D6-PadC2) -> Net-(D6-PadC2)
- D6 pad C3: unconnected-(D6-PadC3) -> GND
- D7 pad A1: unconnected-(D7-PadA1) -> Net-(D6-PadC1)
- D7 pad A2: unconnected-(D7-PadA2) -> Net-(D6-PadC2)
- D7 pad C2: unconnected-(D7-PadC2) -> Net-(D7-PadC2)
- D8 pad A2: unconnected-(D8-PadA2) -> Net-(D7-PadC2)
- D8 pad C1: Net-(D8-PadC1) -> GND
- D8 pad C2: unconnected-(D8-PadC2) -> GND
- D9 pad A1: Net-(D8-PadC1) -> unconnected-(D9-PadA1)

Commit message: cv28 v1.2
Parts:
- added R10: R_Small, Resistor_THT:R_Axial_DIN0617_L17.0mm_D6.0mm_P20.32mm_Horizontal, F.Cu at (795.1, 906.0)
- added R100: R_Small, Resistor_THT:R_Axial_DIN0617_L17.0mm_D6.0mm_P20.32mm_Horizontal, F.Cu at (892.2, 951.2)
- added R101: R_Small, Resistor_THT:R_Axial_DIN0617_L17.0mm_D6.0mm_P20.32mm_Horizontal, F.Cu at (892.2, 958.8)
- added R102: R_Small, Resistor_THT:R_Axial_DIN0617_L17.0mm_D6.0mm_P20.32mm_Horizontal, F.Cu at (892.2, 966.4)
- added R103: R_Small, Resistor_THT:R_Axial_DIN0617_L17.0mm_D6.0mm_P20.32mm_Horizontal, F.Cu at (892.2, 973.9)
- added R104: R_Small, Resistor_THT:R_Axial_DIN0617_L17.0mm_D6.0mm_P20.32mm_Horizontal, F.Cu at (892.2, 981.5)
- added R105: R_Small, Resistor_THT:R_Axial_DIN0617_L17.0mm_D6.0mm_P20.32mm_Horizontal, F.Cu at (892.2, 989.0)
- added R106: R_Small, Resistor_THT:R_Axial_DIN0617_L17.0mm_D6.0mm_P20.32mm_Horizontal, F.Cu at (916.5, 838.0)
- added R107: R_Small, Resistor_THT:R_Axial_DIN0617_L17.0mm_D6.0mm_P20.32mm_Horizontal, F.Cu at (916.5, 845.5)
- added R108: R_Small, Resistor_THT:R_Axial_DIN0617_L17.0mm_D6.0mm_P20.32mm_Horizontal, F.Cu at (916.5, 853.1)
- added R109: R_Small, Resistor_THT:R_Axial_DIN0617_L17.0mm_D6.0mm_P20.32mm_Horizontal, F.Cu at (916.5, 860.6)
- added R11: R_Small, Resistor_THT:R_Axial_DIN0617_L17.0mm_D6.0mm_P20.32mm_Horizontal, F.Cu at (795.1, 913.5)
- added R110: R_Small, Resistor_THT:R_Axial_DIN0617_L17.0mm_D6.0mm_P20.32mm_Horizontal, F.Cu at (916.5, 868.2)
- added R111: R_Small, Resistor_THT:R_Axial_DIN0617_L17.0mm_D6.0mm_P20.32mm_Horizontal, F.Cu at (916.5, 875.8)
- added R112: R_Small, Resistor_THT:R_Axial_DIN0617_L17.0mm_D6.0mm_P20.32mm_Horizontal, F.Cu at (916.5, 883.3)
- added R113: R_Small, Resistor_THT:R_Axial_DIN0617_L17.0mm_D6.0mm_P20.32mm_Horizontal, F.Cu at (916.5, 890.9)
- added R114: R_Small, Resistor_THT:R_Axial_DIN0617_L17.0mm_D6.0mm_P20.32mm_Horizontal, F.Cu at (916.5, 898.4)
- added R115: R_Small, Resistor_THT:R_Axial_DIN0617_L17.0mm_D6.0mm_P20.32mm_Horizontal, F.Cu at (916.5, 906.0)
- added R116: R_Small, Resistor_THT:R_Axial_DIN0617_L17.0mm_D6.0mm_P20.32mm_Horizontal, F.Cu at (916.5, 913.5)
- added R117: R_Small, Resistor_THT:R_Axial_DIN0617_L17.0mm_D6.0mm_P20.32mm_Horizontal, F.Cu at (916.5, 921.0)
- added R118: R_Small, Resistor_THT:R_Axial_DIN0617_L17.0mm_D6.0mm_P20.32mm_Horizontal, F.Cu at (916.5, 928.6)
- added R119: R_Small, Resistor_THT:R_Axial_DIN0617_L17.0mm_D6.0mm_P20.32mm_Horizontal, F.Cu at (916.5, 936.1)
- added R12: R_Small, Resistor_THT:R_Axial_DIN0617_L17.0mm_D6.0mm_P20.32mm_Horizontal, F.Cu at (795.1, 921.0)
- added R120: R_Small, Resistor_THT:R_Axial_DIN0617_L17.0mm_D6.0mm_P20.32mm_Horizontal, F.Cu at (916.5, 943.7)
- added R13: R_Small, Resistor_THT:R_Axial_DIN0617_L17.0mm_D6.0mm_P20.32mm_Horizontal, F.Cu at (795.1, 928.6)
- added R14: R_Small, Resistor_THT:R_Axial_DIN0617_L17.0mm_D6.0mm_P20.32mm_Horizontal, F.Cu at (795.1, 936.1)
- added R15: R_Small, Resistor_THT:R_Axial_DIN0617_L17.0mm_D6.0mm_P20.32mm_Horizontal, F.Cu at (795.1, 943.7)
- added R16: R_Small, Resistor_THT:R_Axial_DIN0617_L17.0mm_D6.0mm_P20.32mm_Horizontal, F.Cu at (795.1, 951.2)
- added R17: R_Small, Resistor_THT:R_Axial_DIN0617_L17.0mm_D6.0mm_P20.32mm_Horizontal, F.Cu at (795.1, 958.8)
- added R18: R_Small, Resistor_THT:R_Axial_DIN0617_L17.0mm_D6.0mm_P20.32mm_Horizontal, F.Cu at (795.1, 966.4)
- added R19: R_Small, Resistor_THT:R_Axial_DIN0617_L17.0mm_D6.0mm_P20.32mm_Horizontal, F.Cu at (795.1, 973.9)
- added R20: R_Small, Resistor_THT:R_Axial_DIN0617_L17.0mm_D6.0mm_P20.32mm_Horizontal, F.Cu at (795.1, 981.5)
- added R21: R_Small, Resistor_THT:R_Axial_DIN0617_L17.0mm_D6.0mm_P20.32mm_Horizontal, F.Cu at (795.1, 989.0)
- added R22: R_Small, Resistor_THT:R_Axial_DIN0617_L17.0mm_D6.0mm_P20.32mm_Horizontal, F.Cu at (819.4, 838.0)
- added R23: R_Small, Resistor_THT:R_Axial_DIN0617_L17.0mm_D6.0mm_P20.32mm_Horizontal, F.Cu at (819.4, 845.5)
- added R24: R_Small, Resistor_THT:R_Axial_DIN0617_L17.0mm_D6.0mm_P20.32mm_Horizontal, F.Cu at (819.4, 853.1)
- added R25: R_Small, Resistor_THT:R_Axial_DIN0617_L17.0mm_D6.0mm_P20.32mm_Horizontal, F.Cu at (819.4, 860.6)
- added R26: R_Small, Resistor_THT:R_Axial_DIN0617_L17.0mm_D6.0mm_P20.32mm_Horizontal, F.Cu at (819.4, 868.2)
- added R27: R_Small, Resistor_THT:R_Axial_DIN0617_L17.0mm_D6.0mm_P20.32mm_Horizontal, F.Cu at (819.4, 875.8)
- added R28: R_Small, Resistor_THT:R_Axial_DIN0617_L17.0mm_D6.0mm_P20.32mm_Horizontal, F.Cu at (819.4, 883.3)
- added R29: R_Small, Resistor_THT:R_Axial_DIN0617_L17.0mm_D6.0mm_P20.32mm_Horizontal, F.Cu at (819.4, 890.9)
- added R30: R_Small, Resistor_THT:R_Axial_DIN0617_L17.0mm_D6.0mm_P20.32mm_Horizontal, F.Cu at (819.4, 898.4)
- added R31: R_Small, Resistor_THT:R_Axial_DIN0617_L17.0mm_D6.0mm_P20.32mm_Horizontal, F.Cu at (819.4, 906.0)
- added R32: R_Small, Resistor_THT:R_Axial_DIN0617_L17.0mm_D6.0mm_P20.32mm_Horizontal, F.Cu at (819.4, 913.5)
- added R33: R_Small, Resistor_THT:R_Axial_DIN0617_L17.0mm_D6.0mm_P20.32mm_Horizontal, F.Cu at (819.4, 921.0)
- added R34: R_Small, Resistor_THT:R_Axial_DIN0617_L17.0mm_D6.0mm_P20.32mm_Horizontal, F.Cu at (819.4, 928.6)
- added R35: R_Small, Resistor_THT:R_Axial_DIN0617_L17.0mm_D6.0mm_P20.32mm_Horizontal, F.Cu at (819.4, 936.1)
- added R36: R_Small, Resistor_THT:R_Axial_DIN0617_L17.0mm_D6.0mm_P20.32mm_Horizontal, F.Cu at (819.4, 943.7)
- added R37: R_Small, Resistor_THT:R_Axial_DIN0617_L17.0mm_D6.0mm_P20.32mm_Horizontal, F.Cu at (819.4, 951.2)
- added R38: R_Small, Resistor_THT:R_Axial_DIN0617_L17.0mm_D6.0mm_P20.32mm_Horizontal, F.Cu at (819.4, 958.8)
- added R39: R_Small, Resistor_THT:R_Axial_DIN0617_L17.0mm_D6.0mm_P20.32mm_Horizontal, F.Cu at (819.4, 966.4)
- added R40: R_Small, Resistor_THT:R_Axial_DIN0617_L17.0mm_D6.0mm_P20.32mm_Horizontal, F.Cu at (819.4, 973.9)
- added R41: R_Small, Resistor_THT:R_Axial_DIN0617_L17.0mm_D6.0mm_P20.32mm_Horizontal, F.Cu at (819.4, 981.5)
- added R42: R_Small, Resistor_THT:R_Axial_DIN0617_L17.0mm_D6.0mm_P20.32mm_Horizontal, F.Cu at (819.4, 989.0)
- added R43: R_Small, Resistor_THT:R_Axial_DIN0617_L17.0mm_D6.0mm_P20.32mm_Horizontal, F.Cu at (843.6, 838.0)
- added R44: R_Small, Resistor_THT:R_Axial_DIN0617_L17.0mm_D6.0mm_P20.32mm_Horizontal, F.Cu at (843.6, 845.5)
- added R45: R_Small, Resistor_THT:R_Axial_DIN0617_L17.0mm_D6.0mm_P20.32mm_Horizontal, F.Cu at (843.6, 853.1)
- added R46: R_Small, Resistor_THT:R_Axial_DIN0617_L17.0mm_D6.0mm_P20.32mm_Horizontal, F.Cu at (843.6, 860.6)
- added R47: R_Small, Resistor_THT:R_Axial_DIN0617_L17.0mm_D6.0mm_P20.32mm_Horizontal, F.Cu at (843.6, 868.2)
- added R48: R_Small, Resistor_THT:R_Axial_DIN0617_L17.0mm_D6.0mm_P20.32mm_Horizontal, F.Cu at (843.6, 875.8)
- added R49: R_Small, Resistor_THT:R_Axial_DIN0617_L17.0mm_D6.0mm_P20.32mm_Horizontal, F.Cu at (843.6, 883.3)
- added R50: R_Small, Resistor_THT:R_Axial_DIN0617_L17.0mm_D6.0mm_P20.32mm_Horizontal, F.Cu at (843.6, 890.9)
- added R51: R_Small, Resistor_THT:R_Axial_DIN0617_L17.0mm_D6.0mm_P20.32mm_Horizontal, F.Cu at (843.6, 898.4)
- added R52: R_Small, Resistor_THT:R_Axial_DIN0617_L17.0mm_D6.0mm_P20.32mm_Horizontal, F.Cu at (843.6, 906.0)
- added R53: R_Small, Resistor_THT:R_Axial_DIN0617_L17.0mm_D6.0mm_P20.32mm_Horizontal, F.Cu at (843.6, 913.5)
- added R54: R_Small, Resistor_THT:R_Axial_DIN0617_L17.0mm_D6.0mm_P20.32mm_Horizontal, F.Cu at (843.6, 921.0)
- added R55: R_Small, Resistor_THT:R_Axial_DIN0617_L17.0mm_D6.0mm_P20.32mm_Horizontal, F.Cu at (843.6, 928.6)
- added R56: R_Small, Resistor_THT:R_Axial_DIN0617_L17.0mm_D6.0mm_P20.32mm_Horizontal, F.Cu at (843.6, 936.1)
- added R57: R_Small, Resistor_THT:R_Axial_DIN0617_L17.0mm_D6.0mm_P20.32mm_Horizontal, F.Cu at (843.6, 943.7)
- added R58: R_Small, Resistor_THT:R_Axial_DIN0617_L17.0mm_D6.0mm_P20.32mm_Horizontal, F.Cu at (843.6, 951.2)
- added R59: R_Small, Resistor_THT:R_Axial_DIN0617_L17.0mm_D6.0mm_P20.32mm_Horizontal, F.Cu at (843.6, 958.8)
- added R60: R_Small, Resistor_THT:R_Axial_DIN0617_L17.0mm_D6.0mm_P20.32mm_Horizontal, F.Cu at (843.6, 966.4)
- added R61: R_Small, Resistor_THT:R_Axial_DIN0617_L17.0mm_D6.0mm_P20.32mm_Horizontal, F.Cu at (843.6, 973.9)
- added R62: R_Small, Resistor_THT:R_Axial_DIN0617_L17.0mm_D6.0mm_P20.32mm_Horizontal, F.Cu at (843.6, 981.5)
- added R63: R_Small, Resistor_THT:R_Axial_DIN0617_L17.0mm_D6.0mm_P20.32mm_Horizontal, F.Cu at (843.6, 989.0)
- added R64: R_Small, Resistor_THT:R_Axial_DIN0617_L17.0mm_D6.0mm_P20.32mm_Horizontal, F.Cu at (867.9, 838.0)
- added R65: R_Small, Resistor_THT:R_Axial_DIN0617_L17.0mm_D6.0mm_P20.32mm_Horizontal, F.Cu at (867.9, 845.5)
- added R66: R_Small, Resistor_THT:R_Axial_DIN0617_L17.0mm_D6.0mm_P20.32mm_Horizontal, F.Cu at (867.9, 853.1)
- added R67: R_Small, Resistor_THT:R_Axial_DIN0617_L17.0mm_D6.0mm_P20.32mm_Horizontal, F.Cu at (867.9, 860.6)
- added R68: R_Small, Resistor_THT:R_Axial_DIN0617_L17.0mm_D6.0mm_P20.32mm_Horizontal, F.Cu at (867.9, 868.2)
- added R69: R_Small, Resistor_THT:R_Axial_DIN0617_L17.0mm_D6.0mm_P20.32mm_Horizontal, F.Cu at (867.9, 875.8)
- added R7: R_Small, Resistor_THT:R_Axial_DIN0617_L17.0mm_D6.0mm_P20.32mm_Horizontal, F.Cu at (795.1, 883.3)
- added R70: R_Small, Resistor_THT:R_Axial_DIN0617_L17.0mm_D6.0mm_P20.32mm_Horizontal, F.Cu at (867.9, 883.3)
- added R71: R_Small, Resistor_THT:R_Axial_DIN0617_L17.0mm_D6.0mm_P20.32mm_Horizontal, F.Cu at (867.9, 890.9)
- added R72: R_Small, Resistor_THT:R_Axial_DIN0617_L17.0mm_D6.0mm_P20.32mm_Horizontal, F.Cu at (867.9, 898.4)
- added R73: R_Small, Resistor_THT:R_Axial_DIN0617_L17.0mm_D6.0mm_P20.32mm_Horizontal, F.Cu at (867.9, 906.0)
- added R74: R_Small, Resistor_THT:R_Axial_DIN0617_L17.0mm_D6.0mm_P20.32mm_Horizontal, F.Cu at (867.9, 913.5)
- added R75: R_Small, Resistor_THT:R_Axial_DIN0617_L17.0mm_D6.0mm_P20.32mm_Horizontal, F.Cu at (867.9, 921.0)
- added R76: R_Small, Resistor_THT:R_Axial_DIN0617_L17.0mm_D6.0mm_P20.32mm_Horizontal, F.Cu at (867.9, 928.6)
- added R77: R_Small, Resistor_THT:R_Axial_DIN0617_L17.0mm_D6.0mm_P20.32mm_Horizontal, F.Cu at (867.9, 936.1)
- added R78: R_Small, Resistor_THT:R_Axial_DIN0617_L17.0mm_D6.0mm_P20.32mm_Horizontal, F.Cu at (867.9, 943.7)
- added R79: R_Small, Resistor_THT:R_Axial_DIN0617_L17.0mm_D6.0mm_P20.32mm_Horizontal, F.Cu at (867.9, 951.2)
- added R8: R_Small, Resistor_THT:R_Axial_DIN0617_L17.0mm_D6.0mm_P20.32mm_Horizontal, F.Cu at (795.1, 890.9)
- added R80: R_Small, Resistor_THT:R_Axial_DIN0617_L17.0mm_D6.0mm_P20.32mm_Horizontal, F.Cu at (867.9, 958.8)
- added R81: R_Small, Resistor_THT:R_Axial_DIN0617_L17.0mm_D6.0mm_P20.32mm_Horizontal, F.Cu at (867.9, 966.4)
- added R82: R_Small, Resistor_THT:R_Axial_DIN0617_L17.0mm_D6.0mm_P20.32mm_Horizontal, F.Cu at (867.9, 973.9)
- added R83: R_Small, Resistor_THT:R_Axial_DIN0617_L17.0mm_D6.0mm_P20.32mm_Horizontal, F.Cu at (867.9, 981.5)
- added R84: R_Small, Resistor_THT:R_Axial_DIN0617_L17.0mm_D6.0mm_P20.32mm_Horizontal, F.Cu at (867.9, 989.0)
- added R85: R_Small, Resistor_THT:R_Axial_DIN0617_L17.0mm_D6.0mm_P20.32mm_Horizontal, F.Cu at (892.2, 838.0)
- added R86: R_Small, Resistor_THT:R_Axial_DIN0617_L17.0mm_D6.0mm_P20.32mm_Horizontal, F.Cu at (892.2, 845.5)
- added R87: R_Small, Resistor_THT:R_Axial_DIN0617_L17.0mm_D6.0mm_P20.32mm_Horizontal, F.Cu at (892.2, 853.1)
- added R88: R_Small, Resistor_THT:R_Axial_DIN0617_L17.0mm_D6.0mm_P20.32mm_Horizontal, F.Cu at (892.2, 860.6)
- added R89: R_Small, Resistor_THT:R_Axial_DIN0617_L17.0mm_D6.0mm_P20.32mm_Horizontal, F.Cu at (892.2, 868.2)
- added R9: R_Small, Resistor_THT:R_Axial_DIN0617_L17.0mm_D6.0mm_P20.32mm_Horizontal, F.Cu at (795.1, 898.4)
- added R90: R_Small, Resistor_THT:R_Axial_DIN0617_L17.0mm_D6.0mm_P20.32mm_Horizontal, F.Cu at (892.2, 875.8)
- added R91: R_Small, Resistor_THT:R_Axial_DIN0617_L17.0mm_D6.0mm_P20.32mm_Horizontal, F.Cu at (892.2, 883.3)
- added R92: R_Small, Resistor_THT:R_Axial_DIN0617_L17.0mm_D6.0mm_P20.32mm_Horizontal, F.Cu at (892.2, 890.9)
- added R93: R_Small, Resistor_THT:R_Axial_DIN0617_L17.0mm_D6.0mm_P20.32mm_Horizontal, F.Cu at (892.2, 898.4)
- added R94: R_Small, Resistor_THT:R_Axial_DIN0617_L17.0mm_D6.0mm_P20.32mm_Horizontal, F.Cu at (892.2, 906.0)
- added R95: R_Small, Resistor_THT:R_Axial_DIN0617_L17.0mm_D6.0mm_P20.32mm_Horizontal, F.Cu at (892.2, 913.5)
- added R96: R_Small, Resistor_THT:R_Axial_DIN0617_L17.0mm_D6.0mm_P20.32mm_Horizontal, F.Cu at (892.2, 921.0)
- added R97: R_Small, Resistor_THT:R_Axial_DIN0617_L17.0mm_D6.0mm_P20.32mm_Horizontal, F.Cu at (892.2, 928.6)
- added R98: R_Small, Resistor_THT:R_Axial_DIN0617_L17.0mm_D6.0mm_P20.32mm_Horizontal, F.Cu at (892.2, 936.1)
- added R99: R_Small, Resistor_THT:R_Axial_DIN0617_L17.0mm_D6.0mm_P20.32mm_Horizontal, F.Cu at (892.2, 943.7)
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Connections:
- D1 pad C1: Net-(D1-PadC1) -> GND
- D1 pad C2: Net-(D1-PadC2) -> GND
- D1 pad C3: Net-(D1-PadC3) -> GND
- D10 pad A1: unconnected-(D10-PadA1) -> Net-(D10-PadA1)
- D10 pad A2: unconnected-(D10-PadA2) -> Net-(D10-PadA2)
- D10 pad A3: unconnected-(D10-PadA3) -> Net-(D10-PadA3)
- D10 pad C1: unconnected-(D10-PadC1) -> Net-(D10-PadC1)
- D10 pad C2: unconnected-(D10-PadC2) -> Net-(D10-PadC2)
- D10 pad C3: unconnected-(D10-PadC3) -> GND
- D100 pad A1: unconnected-(D100-PadA1) -> Net-(D100-PadA1)
- D100 pad A2: unconnected-(D100-PadA2) -> Net-(D100-PadA2)
- D100 pad A3: unconnected-(D100-PadA3) -> Net-(D100-PadA3)
- D100 pad C1: unconnected-(D100-PadC1) -> Net-(D100-PadC1)
- D100 pad C2: unconnected-(D100-PadC2) -> Net-(D100-PadC2)
- D100 pad C3: unconnected-(D100-PadC3) -> GND
- D101 pad A1: unconnected-(D101-PadA1) -> Net-(D101-PadA1)
- D101 pad A2: unconnected-(D101-PadA2) -> Net-(D101-PadA2)
- D101 pad A3: unconnected-(D101-PadA3) -> Net-(D101-PadA3)
- D101 pad C1: unconnected-(D101-PadC1) -> GND
- D101 pad C2: unconnected-(D101-PadC2) -> GND
- D101 pad C3: unconnected-(D101-PadC3) -> Net-(D100-PadA3)
- D102 pad A1: unconnected-(D102-PadA1) -> Net-(D102-PadA1)
- D102 pad A2: unconnected-(D102-PadA2) -> Net-(D102-PadA2)
- D102 pad A3: unconnected-(D102-PadA3) -> Net-(D102-PadA3)
- D102 pad C1: unconnected-(D102-PadC1) -> Net-(D101-PadA1)
- D102 pad C2: unconnected-(D102-PadC2) -> Net-(D101-PadA2)
- D102 pad C3: unconnected-(D102-PadC3) -> Net-(D101-PadA3)
- D103 pad A1: unconnected-(D103-PadA1) -> Net-(D103-PadA1)
- D103 pad A2: unconnected-(D103-PadA2) -> Net-(D103-PadA2)
- D103 pad A3: unconnected-(D103-PadA3) -> Net-(D103-PadA3)
- D103 pad C1: unconnected-(D103-PadC1) -> Net-(D102-PadA1)
- D103 pad C2: unconnected-(D103-PadC2) -> Net-(D102-PadA2)
- D103 pad C3: unconnected-(D103-PadC3) -> GND
- D104 pad A1: unconnected-(D104-PadA1) -> Net-(D104-PadA1)
- D104 pad A2: unconnected-(D104-PadA2) -> Net-(D104-PadA2)
- D104 pad A3: unconnected-(D104-PadA3) -> Net-(D104-PadA3)
- D104 pad C1: unconnected-(D104-PadC1) -> Net-(D103-PadA1)
- D104 pad C2: unconnected-(D104-PadC2) -> Net-(D103-PadA2)
- D104 pad C3: unconnected-(D104-PadC3) -> Net-(D103-PadA3)
- D105 pad A1: unconnected-(D105-PadA1) -> Net-(D105-PadA1)
- D105 pad A2: unconnected-(D105-PadA2) -> Net-(D105-PadA2)
- D105 pad A3: unconnected-(D105-PadA3) -> Net-(D105-PadA3)
- D105 pad C1: unconnected-(D105-PadC1) -> GND
- D105 pad C2: unconnected-(D105-PadC2) -> GND
- D105 pad C3: unconnected-(D105-PadC3) -> Net-(D104-PadA3)
- D106 pad A1: unconnected-(D106-PadA1) -> Net-(D106-PadA1)
- D106 pad A2: unconnected-(D106-PadA2) -> Net-(D106-PadA2)
- D106 pad A3: unconnected-(D106-PadA3) -> Net-(D106-PadA3)
- D106 pad C1: unconnected-(D106-PadC1) -> Net-(D105-PadA1)
- D106 pad C2: unconnected-(D106-PadC2) -> Net-(D105-PadA2)
- D106 pad C3: unconnected-(D106-PadC3) -> GND
- D107 pad A1: unconnected-(D107-PadA1) -> Net-(D107-PadA1)
- D107 pad A2: unconnected-(D107-PadA2) -> Net-(D107-PadA2)
- D107 pad A3: unconnected-(D107-PadA3) -> Net-(D107-PadA3)
- D107 pad C1: unconnected-(D107-PadC1) -> Net-(D106-PadA1)
- D107 pad C2: unconnected-(D107-PadC2) -> Net-(D106-PadA2)
- D107 pad C3: unconnected-(D107-PadC3) -> Net-(D106-PadA3)
- D108 pad A1: unconnected-(D108-PadA1) -> Net-(D108-PadA1)
- D108 pad A2: unconnected-(D108-PadA2) -> Net-(D108-PadA2)
- D108 pad A3: unconnected-(D108-PadA3) -> Net-(D108-PadA3)
- D108 pad C1: unconnected-(D108-PadC1) -> Net-(D107-PadA1)
- D108 pad C2: unconnected-(D108-PadC2) -> Net-(D107-PadA2)
- D108 pad C3: unconnected-(D108-PadC3) -> Net-(D107-PadA3)
- D109 pad A1: unconnected-(D109-PadA1) -> Net-(D109-PadA1)
- D109 pad A2: unconnected-(D109-PadA2) -> Net-(D109-PadA2)
- D109 pad A3: unconnected-(D109-PadA3) -> Net-(D109-PadA3)
- D109 pad C1: unconnected-(D109-PadC1) -> GND
- D109 pad C2: unconnected-(D109-PadC2) -> GND
- D109 pad C3: unconnected-(D109-PadC3) -> GND
- D11 pad A1: unconnected-(D11-PadA1) -> Net-(D11-PadA1)
- D11 pad A2: unconnected-(D11-PadA2) -> Net-(D11-PadA2)
- D11 pad A3: unconnected-(D11-PadA3) -> Net-(D11-PadA3)
- D11 pad C1: unconnected-(D11-PadC1) -> Net-(D10-PadA1)
- D11 pad C2: unconnected-(D11-PadC2) -> Net-(D10-PadA2)
- D11 pad C3: unconnected-(D11-PadC3) -> Net-(D10-PadA3)
- D110 pad A1: unconnected-(D110-PadA1) -> Net-(D110-PadA1)
- D110 pad A2: unconnected-(D110-PadA2) -> Net-(D110-PadA2)
- D110 pad A3: unconnected-(D110-PadA3) -> Net-(D110-PadA3)
- D110 pad C1: unconnected-(D110-PadC1) -> Net-(D109-PadA1)
- D110 pad C2: unconnected-(D110-PadC2) -> Net-(D109-PadA2)
- D110 pad C3: unconnected-(D110-PadC3) -> Net-(D109-PadA3)
- D111 pad A1: unconnected-(D111-PadA1) -> Net-(D111-PadA1)
- D111 pad A2: unconnected-(D111-PadA2) -> Net-(D111-PadA2)
- D111 pad A3: unconnected-(D111-PadA3) -> Net-(D111-PadA3)
- D111 pad C1: unconnected-(D111-PadC1) -> Net-(D110-PadA1)
- D111 pad C2: unconnected-(D111-PadC2) -> Net-(D110-PadA2)
- D111 pad C3: unconnected-(D111-PadC3) -> Net-(D110-PadA3)
- D112 pad A1: unconnected-(D112-PadA1) -> Net-(D112-PadA1)
- D112 pad A2: unconnected-(D112-PadA2) -> Net-(D112-PadA2)
- D112 pad A3: unconnected-(D112-PadA3) -> Net-(D112-PadA3)
- D112 pad C1: unconnected-(D112-PadC1) -> Net-(D111-PadA1)
- D112 pad C2: unconnected-(D112-PadC2) -> Net-(D111-PadA2)
- D112 pad C3: unconnected-(D112-PadC3) -> GND
- D113 pad A1: unconnected-(D113-PadA1) -> Net-(D113-PadA1)
- D113 pad A2: unconnected-(D113-PadA2) -> Net-(D113-PadA2)
- D113 pad A3: unconnected-(D113-PadA3) -> Net-(D113-PadA3)
- D113 pad C1: unconnected-(D113-PadC1) -> GND
- D113 pad C2: unconnected-(D113-PadC2) -> GND
- D113 pad C3: unconnected-(D113-PadC3) -> Net-(D112-PadA3)
- D114 pad A1: unconnected-(D114-PadA1) -> Net-(D114-PadA1)
- D114 pad A2: unconnected-(D114-PadA2) -> Net-(D114-PadA2)
- D114 pad A3: unconnected-(D114-PadA3) -> Net-(D114-PadA3)
- D114 pad C1: unconnected-(D114-PadC1) -> Net-(D113-PadA1)
- D114 pad C2: unconnected-(D114-PadC2) -> Net-(D113-PadA2)
- D114 pad C3: unconnected-(D114-PadC3) -> Net-(D113-PadA3)
- D115 pad A1: unconnected-(D115-PadA1) -> Net-(D115-PadA1)
- D115 pad A2: unconnected-(D115-PadA2) -> Net-(D115-PadA2)
- D115 pad A3: unconnected-(D115-PadA3) -> Net-(D115-PadA3)
- D115 pad C1: unconnected-(D115-PadC1) -> Net-(D114-PadA1)
- D115 pad C2: unconnected-(D115-PadC2) -> Net-(D114-PadA2)
- D115 pad C3: unconnected-(D115-PadC3) -> GND
- D116 pad A1: unconnected-(D116-PadA1) -> Net-(D116-PadA1)
- D116 pad A2: unconnected-(D116-PadA2) -> Net-(D116-PadA2)
- D116 pad A3: unconnected-(D116-PadA3) -> Net-(D116-PadA3)
- D116 pad C1: unconnected-(D116-PadC1) -> Net-(D115-PadA1)
- D116 pad C2: unconnected-(D116-PadC2) -> Net-(D115-PadA2)
- D116 pad C3: unconnected-(D116-PadC3) -> Net-(D115-PadA3)
- D117 pad A1: unconnected-(D117-PadA1) -> Net-(D117-PadA1)
- D117 pad A2: unconnected-(D117-PadA2) -> Net-(D117-PadA2)
- D117 pad A3: unconnected-(D117-PadA3) -> Net-(D117-PadA3)
- D117 pad C1: unconnected-(D117-PadC1) -> GND
- D117 pad C2: unconnected-(D117-PadC2) -> GND
- D117 pad C3: unconnected-(D117-PadC3) -> Net-(D116-PadA3)
- D118 pad A1: unconnected-(D118-PadA1) -> Net-(D118-PadA1)
- D118 pad A2: unconnected-(D118-PadA2) -> Net-(D118-PadA2)
- D118 pad A3: unconnected-(D118-PadA3) -> Net-(D118-PadA3)
- D118 pad C1: unconnected-(D118-PadC1) -> Net-(D117-PadA1)
- D118 pad C2: unconnected-(D118-PadC2) -> Net-(D117-PadA2)
- D118 pad C3: unconnected-(D118-PadC3) -> GND
- D119 pad A1: unconnected-(D119-PadA1) -> Net-(D119-PadA1)
- D119 pad A2: unconnected-(D119-PadA2) -> Net-(D119-PadA2)
- D119 pad A3: unconnected-(D119-PadA3) -> Net-(D119-PadA3)
- D119 pad C1: unconnected-(D119-PadC1) -> Net-(D118-PadA1)
- D119 pad C2: unconnected-(D119-PadC2) -> Net-(D118-PadA2)
- D119 pad C3: unconnected-(D119-PadC3) -> Net-(D118-PadA3)
- D12 pad A1: unconnected-(D12-PadA1) -> Net-(D12-PadA1)
- D12 pad A2: unconnected-(D12-PadA2) -> Net-(D12-PadA2)
- D12 pad A3: unconnected-(D12-PadA3) -> Net-(D12-PadA3)
- D12 pad C1: unconnected-(D12-PadC1) -> Net-(D11-PadA1)
- D12 pad C2: unconnected-(D12-PadC2) -> Net-(D11-PadA2)
- D12 pad C3: unconnected-(D12-PadC3) -> Net-(D11-PadA3)
- D120 pad A1: unconnected-(D120-PadA1) -> Net-(D120-PadA1)
- D120 pad A2: unconnected-(D120-PadA2) -> Net-(D120-PadA2)
- D120 pad A3: unconnected-(D120-PadA3) -> Net-(D120-PadA3)
- D120 pad C1: unconnected-(D120-PadC1) -> Net-(D119-PadA1)
- D120 pad C2: unconnected-(D120-PadC2) -> Net-(D119-PadA2)
- D120 pad C3: unconnected-(D120-PadC3) -> Net-(D119-PadA3)
- D121 pad A1: unconnected-(D121-PadA1) -> Net-(D121-PadA1)
- D121 pad A2: unconnected-(D121-PadA2) -> Net-(D121-PadA2)
- D121 pad A3: unconnected-(D121-PadA3) -> Net-(D121-PadA3)
- D121 pad C1: unconnected-(D121-PadC1) -> GND
- D121 pad C2: unconnected-(D121-PadC2) -> GND
- D121 pad C3: unconnected-(D121-PadC3) -> GND
- D122 pad A1: unconnected-(D122-PadA1) -> Net-(D122-PadA1)
- D122 pad A2: unconnected-(D122-PadA2) -> Net-(D122-PadA2)
- D122 pad A3: unconnected-(D122-PadA3) -> Net-(D122-PadA3)
- D122 pad C1: unconnected-(D122-PadC1) -> Net-(D121-PadA1)
- D122 pad C2: unconnected-(D122-PadC2) -> Net-(D121-PadA2)
- D122 pad C3: unconnected-(D122-PadC3) -> Net-(D121-PadA3)
- D123 pad A1: unconnected-(D123-PadA1) -> Net-(D123-PadA1)
- D123 pad A2: unconnected-(D123-PadA2) -> Net-(D123-PadA2)
- D123 pad A3: unconnected-(D123-PadA3) -> Net-(D123-PadA3)
- D123 pad C1: unconnected-(D123-PadC1) -> Net-(D122-PadA1)
- D123 pad C2: unconnected-(D123-PadC2) -> Net-(D122-PadA2)
- D123 pad C3: unconnected-(D123-PadC3) -> Net-(D122-PadA3)
- D124 pad A1: unconnected-(D124-PadA1) -> Net-(D124-PadA1)
- D124 pad A2: unconnected-(D124-PadA2) -> Net-(D124-PadA2)
- D124 pad A3: unconnected-(D124-PadA3) -> Net-(D124-PadA3)
- D124 pad C1: unconnected-(D124-PadC1) -> Net-(D123-PadA1)
- D124 pad C2: unconnected-(D124-PadC2) -> Net-(D123-PadA2)
- D124 pad C3: unconnected-(D124-PadC3) -> GND
- D125 pad A1: unconnected-(D125-PadA1) -> Net-(D125-PadA1)
- D125 pad A2: unconnected-(D125-PadA2) -> Net-(D125-PadA2)
- D125 pad A3: unconnected-(D125-PadA3) -> Net-(D125-PadA3)
- D125 pad C1: unconnected-(D125-PadC1) -> GND
- D125 pad C2: unconnected-(D125-PadC2) -> GND
- D125 pad C3: unconnected-(D125-PadC3) -> Net-(D124-PadA3)
- D126 pad A1: unconnected-(D126-PadA1) -> Net-(D126-PadA1)
- D126 pad A2: unconnected-(D126-PadA2) -> Net-(D126-PadA2)
- D126 pad A3: unconnected-(D126-PadA3) -> Net-(D126-PadA3)
- D126 pad C1: unconnected-(D126-PadC1) -> Net-(D125-PadA1)
- D126 pad C2: unconnected-(D126-PadC2) -> Net-(D125-PadA2)
- D126 pad C3: unconnected-(D126-PadC3) -> Net-(D125-PadA3)
- D127 pad A1: unconnected-(D127-PadA1) -> Net-(D127-PadA1)
- D127 pad A2: unconnected-(D127-PadA2) -> Net-(D127-PadA2)
- D127 pad A3: unconnected-(D127-PadA3) -> Net-(D127-PadA3)
- D127 pad C1: unconnected-(D127-PadC1) -> Net-(D126-PadA1)
- D127 pad C2: unconnected-(D127-PadC2) -> Net-(D126-PadA2)
- D127 pad C3: unconnected-(D127-PadC3) -> GND
- D128 pad A1: unconnected-(D128-PadA1) -> Net-(D128-PadA1)
- D128 pad A2: unconnected-(D128-PadA2) -> Net-(D128-PadA2)
- D128 pad A3: unconnected-(D128-PadA3) -> Net-(D128-PadA3)
- D128 pad C1: unconnected-(D128-PadC1) -> Net-(D127-PadA1)
- D128 pad C2: unconnected-(D128-PadC2) -> Net-(D127-PadA2)
- D128 pad C3: unconnected-(D128-PadC3) -> Net-(D127-PadA3)
- D129 pad A1: unconnected-(D129-PadA1) -> Net-(D129-PadA1)
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
Commit message: cv28 v1.3
Parts:
- R1: renamed from R10; footprint Resistor_THT:R_Axial_DIN0617_L17.0mm_D6.0mm_P20.32mm_Horizontal -> Resistor_THT:R_Axial_DIN0207_L6.3mm_D2.5mm_P10.16mm_Horizontal
- R10: renamed from R3; footprint Resistor_THT:R_Axial_DIN0617_L17.0mm_D6.0mm_P20.32mm_Horizontal -> Resistor_THT:R_Axial_DIN0207_L6.3mm_D2.5mm_P10.16mm_Horizontal
- R100, R101, R102, R103, R104, R105, R106, R107, R108, R109, R11, R110, R111, R112, R113, R114, R115, R116, R117, R118, R119, R12, R120, R13, R14, R15, R16, R17, R18, R19, R20, R21, R22, R23, R24, R25, R26, R27, R28, R29, R30, R31, R32, R33, R34, R35, R36, R37, R38, R39, R40, R41, R42, R43, R44, R45, R46, R47, R48, R49, R50, R51, R52, R53, R54, R55, R56, R57, R58, R59, R60, R61, R62, R63, R64, R65, R66, R67, R68, R69, R70, R71, R72, R73, R74, R75, R76, R77, R78, R79, R80, R81, R82, R83, R84, R85, R86, R87, R88, R89, R90, R91, R92, R93, R94, R95, R96, R97, R98, R99: footprint Resistor_THT:R_Axial_DIN0617_L17.0mm_D6.0mm_P20.32mm_Horizontal -> Resistor_THT:R_Axial_DIN0207_L6.3mm_D2.5mm_P10.16mm_Horizontal
- R2: renamed from R7; footprint Resistor_THT:R_Axial_DIN0617_L17.0mm_D6.0mm_P20.32mm_Horizontal -> Resistor_THT:R_Axial_DIN0207_L6.3mm_D2.5mm_P10.16mm_Horizontal
- R3: renamed from R8; footprint Resistor_THT:R_Axial_DIN0617_L17.0mm_D6.0mm_P20.32mm_Horizontal -> Resistor_THT:R_Axial_DIN0207_L6.3mm_D2.5mm_P10.16mm_Horizontal
- R4: renamed from R9; footprint Resistor_THT:R_Axial_DIN0617_L17.0mm_D6.0mm_P20.32mm_Horizontal -> Resistor_THT:R_Axial_DIN0207_L6.3mm_D2.5mm_P10.16mm_Horizontal
- R5: renamed from R4; footprint Resistor_THT:R_Axial_DIN0617_L17.0mm_D6.0mm_P20.32mm_Horizontal -> Resistor_THT:R_Axial_DIN0207_L6.3mm_D2.5mm_P10.16mm_Horizontal
- R6: renamed from R5; footprint Resistor_THT:R_Axial_DIN0617_L17.0mm_D6.0mm_P20.32mm_Horizontal -> Resistor_THT:R_Axial_DIN0207_L6.3mm_D2.5mm_P10.16mm_Horizontal
- R7: renamed from R6; footprint Resistor_THT:R_Axial_DIN0617_L17.0mm_D6.0mm_P20.32mm_Horizontal -> Resistor_THT:R_Axial_DIN0207_L6.3mm_D2.5mm_P10.16mm_Horizontal
- R8: renamed from R1; footprint Resistor_THT:R_Axial_DIN0617_L17.0mm_D6.0mm_P20.32mm_Horizontal -> Resistor_THT:R_Axial_DIN0207_L6.3mm_D2.5mm_P10.16mm_Horizontal
- R9: renamed from R2; footprint Resistor_THT:R_Axial_DIN0617_L17.0mm_D6.0mm_P20.32mm_Horizontal -> Resistor_THT:R_Axial_DIN0207_L6.3mm_D2.5mm_P10.16mm_Horizontal
- moved R61 1009.1 mm to (194.6, 201.3)
- moved R62 1009.0 mm to (194.6, 208.9)
- moved R63 1008.9 mm to (194.7, 216.6)
- moved D74 982.3 mm to (277.3, 157.5)
- moved R60 970.8 mm to (360.1, 124.5), turned to -90 degrees
- moved D73 968.8 mm to (292.8, 157.5)
- moved D75 966.5 mm to (259.7, 202.2)
- moved R59 960.5 mm to (367.7, 124.5), turned to -90 degrees
- moved D72 955.4 mm to (308.4, 157.3)
- moved D76 950.7 mm to (270.6, 217.3)
- moved R58 950.2 mm to (375.4, 124.5), turned to -90 degrees
- moved D68 946.7 mm to (370.4, 157.3)
- moved D71 942.2 mm to (323.9, 157.1)
- moved R57 939.8 mm to (383.0, 124.5), turned to -90 degrees
- moved D77 935.0 mm to (281.5, 232.5)
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