File: Chevron_signal.kicad_sch (KiCad schematic)
At the start: 30 parts

Commit message: cv28 v1.0
Parts:
- removed D1, D10, D11, D12, D13, D14, D15, D16, D17, D18, D19, D2, D20, D21, D22, D23, D24, D25, D26, D27, D28, D29, D3, D30, D4, D5, D6, D7, D8, D9: L08R5000Q1, L08R5000Q1:LEDRD254W57D500H1070, symbol L08R5000Q1:L08R5000Q1
- added D1, D10, D11, D12, D13, D14, D15, D16, D17, D18, D19, D2, D20, D21, D22, D23, D24, D3, D4, D5, D6, D7, D8, D9: LED_CV28, LED_CV28, symbol LED_CV28:LED_CV28
Connections:
- new net: D20.C1, D21.A1
- new net: D11.C1, D12.A1
- new net: D4.C1, D5.A1
- new net: D5.C1, D6.A1
- new net: D17.C1, D18.A1
- new net: D2.C1, D3.A1
- new net: D13.C1, D14.A1
- new net: D14.C1, D15.A1
- new net: D7.C1, D8.A1
- new net: D8.C1, D9.A1
- new net: D22.C1, D23.A1
- new net: D16.C1, D17.A1
- new net: D19.C1, D20.A1
- new net: D10.C1, D11.A1
- new net: D1.C1, D2.A1
- new net: D23.C1, D24.A1

Commit message: cv28 v1.1
Parts:
- added D100, D101, D102, D103, D104, D105, D106, D107, D108, D109, D110, D111, D112, D113, D114, D115, D116, D117, D118, D119, D120, D121, D122, D123, D124, D125, D126, D127, D128, D129, D130, D131, D132, D133, D134, D135, D136, D137, D138, D139, D140, D141, D142, D143, D144, D25, D26, D27, D28, D29, D30, D31, D32, D33, D34, D35, D36, D37, D38, D39, D40, D41, D42, D43, D44, D45, D46, D47, D48, D49, D50, D51, D52, D53, D54, D55, D56, D57, D58, D59, D60, D61, D62, D63, D64, D65, D66, D67, D68, D69, D70, D71, D72, D73, D74, D75, D76, D77, D78, D79, D80, D81, D82, D83, D84, D85, D86, D87, D88, D89, D90, D91, D92, D93, D94, D95, D96, D97, D98, D99: LED_CV28, LED_CV28, symbol LED_CV28:LED_CV28
- added P1: 282837-2, 282837-2:TE_282837-2, symbol 282837-2:282837-2
- added R1, R10, R2, R3, R4, R5, R6, R7, R8, R9: R_Small, Resistor_THT:R_Axial_DIN0617_L17.0mm_D6.0mm_P20.32mm_Horizontal, symbol Device:R_Small
Connections:
- net at D21.A1: no longer D20.C1
- net at D12.A2: now also D11.C2
- net at D12.A3: now also D11.C3
- net GND: now reaches D12.C1
- net GND: now also D12.C2, D12.C3, D3.C3, D4.C1, D4.C2, D6.C3, D8.C1, D8.C2, D9.C3
- net at D5.A1: now also R10.2, R4.1, R7.2, R8.2, R9.2; no longer D4.C1
- net at D5.A2: now also R5.1
- net at D5.A3: now also D4.C3
- net at D5.C2: now also D6.A2
- net at D5.C3: now also D6.A3
- net at D18.A1: no longer D17.C1
- net at D3.A2: now also D2.C2
- net at D3.A3: now also D2.C3
- net at D3.C1: now also D4.A1
- net at D3.C2: now also D4.A2
- net at D13.C1: no longer D14.A1
- net at D14.C1: no longer D15.A1
- net at D7.A1: now also D6.C1
- net at D7.A2: now also D6.C2
- net at D7.A3: now also R9.1
- net at D7.C2: now also D8.A2
- net at D7.C3: now also D8.A3
- net at D9.A1: now also R7.1; no longer D8.C1
- net at D8.C3: now also D9.A3
- net at D22.C1: no longer D23.A1
- net at D17.A1: no longer D16.C1
- net at D4.A3: now also R6.1
- net at D19.C1: no longer D20.A1
- net at D10.A1: now also D9.C1
- net at D10.A2: now also D9.C2
- net at D10.A3: now also R10.1
- net at D10.C2: now also D11.A2
- net at D10.C3: now also D11.A3
- net at D2.A2: now also D1.C2
- net at D2.A3: now also D1.C3
- net at D23.C1: no longer D24.A1
- net at D1.A1: now also R1.1
- net at D1.A2: now also R2.1
- net at D1.A3: now also R3.1
- net at D9.A2: now also R8.1
- new net: R4.2, R5.2, R6.2
- new net +12V: R1.2, R2.2, R3.2
Other:
- moved on the sheet: D1, D10, D11, D12, D13, D14, D15, D16, D17, D18, D19, D2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

Commit message: cv28 v1.2
Parts:
- added R100, R101, R102, R103, R104, R105, R106, R107, R108, R109, R11, R110, R111, R112, R113, R114, R115, R116, R117, R118, R119, R12, R120, R13, R14, R15, R16, R17, R18, R19, R20, R21, R22, R23, R24, R25, R26, R27, R28, R29, R30, R31, R32, R33, R34, R35, R36, R37, R38, R39, R40, R41, R42, R43, R44, R45, R46, R47, R48, R49, R50, R51, R52, R53, R54, R55, R56, R57, R58, R59, R60, R61, R62, R63, R64, R65, R66, R67, R68, R69, R70, R71, R72, R73, R74, R75, R76, R77, R78, R79, R80, R81, R82, R83, R84, R85, R86, R87, R88, R89, R90, R91, R92, R93, R94, R95, R96, R97, R98, R99: R_Small, Resistor_THT:R_Axial_DIN0617_L17.0mm_D6.0mm_P20.32mm_Horizontal, symbol Device:R_Small
- renumbered D12 to D1, D3 to D10, D2 to D11, D1 to D12, D11 to D2, D10 to D3, D9 to D4, D8 to D5, D7 to D6, D6 to D7, D5 to D8, D4 to D9
Connections:
- net +12V: now also P1.2, R10.2, R4.2, R5.2, R6.2, R7.2, R8.2, R9.2, R100.2, R101.2, R102.2, R103.2, R104.2, R105.2, R106.2, R107.2, R108.2, R109.2, R11.2, R110.2, R111.2, R112.2, R113.2, R114.2, R115.2, R116.2, R117.2, R118.2, R119.2, R12.2, R120.2, R13.2, R14.2, R15.2, R16.2, R17.2, R18.2, R19.2, R20.2, R21.2, R22.2, R23.2, R24.2, R25.2, R26.2, R27.2, R28.2, R29.2, R30.2, R31.2, R32.2, R33.2, R34.2, R35.2, R36.2, R37.2, R38.2, R39.2, R40.2, R41.2, R42.2, R43.2, R44.2, R45.2, R46.2, R47.2, R48.2, R49.2, R50.2, R51.2, R52.2, R53.2, R54.2, R55.2, R56.2, R57.2, R58.2, R59.2, R60.2, R61.2, R62.2, R63.2, R64.2, R65.2, R66.2, R67.2, R68.2, R69.2, R70.2, R71.2, R72.2, R73.2, R74.2, R75.2, R76.2, R77.2, R78.2, R79.2, R80.2, R81.2, R82.2, R83.2, R84.2, R85.2, R86.2, R87.2, R88.2, R89.2, R90.2, R91.2, R92.2, R93.2, R94.2, R95.2, R96.2, R97.2, R98.2, R99.2
- net GND: now also D100.C3, D101.C1, D101.C2, D103.C3, D105.C1, D105.C2, D106.C3, D109.C1, D109.C2, D109.C3, D112.C3, D113.C1, D113.C2, D115.C3, D117.C1, D117.C2, D118.C3, D121.C1, D121.C2, D121.C3, D124.C3, D125.C1, D125.C2, D127.C3, D129.C1, D129.C2, D13.C1, D13.C2, D13.C3, D130.C3, D133.C1, D133.C2, D133.C3, D136.C3, D137.C1, D137.C2, D139.C3, D141.C1, D141.C2, D142.C3, D16.C3, D17.C1, D17.C2, D19.C3, D21.C1, D21.C2, D22.C3, D25.C1, D25.C2, D25.C3, D28.C3, D29.C1, D29.C2, D31.C3, D33.C1, D33.C2, D34.C3, D37.C1, D37.C2, D37.C3, D40.C3, D41.C1, D41.C2, D43.C3, D45.C1, D45.C2, D46.C3, D49.C1, D49.C2, D49.C3, D52.C3, D53.C1, D53.C2, D55.C3, D57.C1, D57.C2, D58.C3, D61.C1, D61.C2, D61.C3, D64.C3, D65.C1, D65.C2, D67.C3, D69.C1, D69.C2, D70.C3, D73.C1, D73.C2, D73.C3, D76.C3, D77.C1, D77.C2, D79.C3, D81.C1, D81.C2, D82.C3, D85.C1, D85.C2, D85.C3, D88.C3, D89.C1, D89.C2, D91.C3, D93.C1, D93.C2, D94.C3, D97.C1, D97.C2, D97.C3, P1.1
- net at D119.A1: now also D120.C1
- net at D119.A2: now also D120.C2
- net at D119.A3: now also D120.C3
- net at D119.C1: now also D118.A1
- net at D119.C2: now also D118.A2
- net at D119.C3: now also D118.A3
- net at D91.A1: now also D92.C1
- net at D91.A2: now also D92.C2
- net at D91.A3: now also D92.C3
- net at D91.C1: now also D90.A1
- net at D91.C2: now also D90.A2
- net at D126.A1: now also D127.C1
- net at D126.A2: now also D127.C2
- net at D126.A3: now also R104.1
- net at D126.C1: now also D125.A1
- net at D126.C2: now also D125.A2
- net at D126.C3: now also D125.A3
- net at D122.A1: now also D123.C1
- net at D122.A2: now also D123.C2
- net at D122.A3: now also D123.C3
- net at D122.C1: now also D121.A1
- net at D122.C2: now also D121.A2
- net at D122.C3: now also D121.A3
- net at D21.A1: now also D22.C1
- net at D21.A2: now also D22.C2
- net at D21.A3: now also R17.1
- net at D21.C3: now also D20.A3
- net at D136.A1: now also R112.1
- net at D136.A2: now also R113.1
- net at D136.A3: now also D137.C3
- net at D136.C1: now also D135.A1
- net at D136.C2: now also D135.A2
- net at D137.A1: now also D138.C1
- net at D137.A2: now also D138.C2
- net at D137.A3: now also D138.C3
- net at D28.A1: now also R22.1
- net at D28.A2: now also R23.1
- net at D28.A3: now also D29.C3
- net at D28.C1: now also D27.A1
- net at D28.C2: now also D27.A2
- net at D67.A1: now also D68.C1
- net at D67.A2: now also D68.C2
- net at D67.A3: now also D68.C3
- net at D67.C1: now also D66.A1
- net at D67.C2: now also D66.A2
- net at D38.A1: now also D39.C1
- net at D38.A2: now also D39.C2
- net at D38.A3: now also D39.C3
- net at D38.C1: now also D37.A1
- net at D38.C2: now also D37.A2
- net at D38.C3: now also D37.A3
- net at D87.A1: now also D88.C1
- net at D87.A2: now also D88.C2
- net at D87.A3: now also R71.1
- net at D87.C1: now also D86.A1
- net at D87.C2: now also D86.A2
- net at D87.C3: now also D86.A3
- net at D97.A1: now also D98.C1
- net at D97.A2: now also D98.C2
- net at D97.A3: now also D98.C3
- net at D117.A1: now also D118.C1
- net at D117.A2: now also D118.C2
- net at D117.A3: now also R97.1
- net at D117.C3: now also D116.A3
- net at D112.A1: now also R92.1
- net at D112.A2: now also R93.1
- net at D112.A3: now also D113.C3
- net at D112.C1: now also D111.A1
- net at D112.C2: now also D111.A2
- net at D79.A1: now also D80.C1
- net at D79.A2: now also D80.C2
- net at D79.A3: now also D80.C3
- net at D79.C1: now also D78.A1
- net at D79.C2: now also D78.A2
- net at D47.A1: now also D48.C1
- net at D47.A2: now also D48.C2
- net at D47.A3: now also D48.C3
- net at D47.C1: now also D46.A1
- net at D47.C2: now also D46.A2
- net at D47.C3: now also D46.A3
- net at D69.A1: now also D70.C1
- net at D69.A2: now also D70.C2
- net at D69.A3: now also R57.1
- net at D69.C3: now also D68.A3
- net at D39.A1: now also D40.C1
- net at D39.A2: now also D40.C2
- net at D39.A3: now also R31.1
- net at D18.A1: now also D19.C1
- net at D18.A2: now also D19.C2
- net at D18.A3: now also R14.1
- net at D18.C1: now also D17.A1
- net at D18.C2: now also D17.A2
- net at D18.C3: now also D17.A3
- net at D35.A1: now also D36.C1
- net at D35.A2: now also D36.C2
- net at D35.A3: now also D36.C3
- net at D35.C1: now also D34.A1
- net at D35.C2: now also D34.A2
- net at D35.C3: now also D34.A3
- net at D108.A1: now also R88.1
- net at D108.A2: now also R89.1
- net at D108.A3: now also R90.1
- net at D108.C1: now also D107.A1
- net at D108.C2: now also D107.A2
- net at D108.C3: now also D107.A3
- net at D51.A1: now also D52.C1
- net at D51.A2: now also D52.C2
- net at D51.A3: now also R41.1
- net at D51.C1: now also D50.A1
- net at D51.C2: now also D50.A2
- net at D51.C3: now also D50.A3
- net at D77.A1: now also D78.C1
- net at D77.A2: now also D78.C2
- net at D77.A3: now also D78.C3
- net at D77.C3: now also D76.A3
- net at D13.A1: now also D14.C1
- net at D13.A2: now also D14.C2
- net at D13.A3: now also D14.C3
- net at D50.C1: now also D49.A1
- net at D50.C2: now also D49.A2
- net at D50.C3: now also D49.A3
- net at D53.A1: now also D54.C1
- net at D53.A2: now also D54.C2
- net at D53.A3: now also D54.C3
- net at D53.C3: now also D52.A3
- net at D14.A1: now also D15.C1
- net at D14.A2: now also D15.C2
- net at D14.A3: now also D15.C3
- net at D68.A1: now also R55.1
- net at D68.A2: now also R56.1
- net at D52.A1: now also R42.1
- net at D52.A2: now also R43.1
- net at D65.A1: now also D66.C1
- net at D65.A2: now also D66.C2
- net at D65.A3: now also D66.C3
- net at D65.C3: now also D64.A3
- net at D26.A1: now also D27.C1
- net at D26.A2: now also D27.C2
- net at D26.A3: now also D27.C3
- net at D26.C1: now also D25.A1
- net at D26.C2: now also D25.A2
- net at D26.C3: now also D25.A3
- net at D15.A1: now also D16.C1
- net at D15.A2: now also D16.C2
- net at D15.A3: now also R11.1
- net at D22.A1: now also D23.C1
- net at D22.A2: now also D23.C2
- net at D22.A3: now also D23.C3
- net at D27.A3: now also R21.1
- net at D31.A1: now also D32.C1
- net at D31.A2: now also D32.C2
- net at D31.A3: now also D32.C3
- net at D31.C1: now also D30.A1
- net at D31.C2: now also D30.A2
- net at D41.A1: now also D42.C1
- net at D41.A2: now also D42.C2
- net at D41.A3: now also D42.C3
- net at D41.C3: now also D40.A3
- net at D17.C3: now also D16.A3
- net at D124.A1: now also R102.1
- net at D124.A2: now also R103.1
- net at D124.A3: now also D125.C3
- net at D124.C1: now also D123.A1
- net at D124.C2: now also D123.A2
- net at D82.A1: now also D83.C1
- net at D82.A2: now also D83.C2
- net at D82.A3: now also D83.C3
- net at D82.C1: now also D81.A1
- net at D82.C2: now also D81.A2
- net at D42.A1: now also D43.C1
- net at D42.A2: now also D43.C2
- net at D42.A3: now also R34.1
- net at D142.A1: now also D143.C1
- net at D142.A2: now also D143.C2
- net at D142.A3: now also D143.C3
- net at D142.C1: now also D141.A1
- net at D142.C2: now also D141.A2
- net at D29.A1: now also D30.C1
- net at D29.A2: now also D30.C2
- net at D29.A3: now also D30.C3
- net at D120.A1: now also R98.1
- net at D120.A2: now also R99.1
- net at D120.A3: now also R100.1
- net at D78.A3: now also R64.1
- net at D60.A1: now also R48.1
- net at D60.A2: now also R49.1
- net at D60.A3: now also R50.1
- net at D60.C1: now also D59.A1
- net at D60.C2: now also D59.A2
- net at D60.C3: now also D59.A3
- net at D66.A3: now also R54.1
- net at D133.A1: now also D134.C1
- net at D133.A2: now also D134.C2
- net at D133.A3: now also D134.C3
- net at D19.A1: now also D20.C1
- net at D19.A2: now also D20.C2
- net at D19.A3: now also D20.C3
- net at D83.A1: now also D84.C1
- net at D83.A2: now also D84.C2
- net at D83.A3: now also D84.C3
- net at D110.A1: now also D111.C1
- net at D110.A2: now also D111.C2
- net at D110.A3: now also D111.C3
- net at D110.C1: now also D109.A1
- net at D110.C2: now also D109.A2
- net at D110.C3: now also D109.A3
- net at D106.A1: now also D107.C1
- net at D106.A2: now also D107.C2
- net at D106.A3: now also D107.C3
- net at D106.C1: now also D105.A1
- net at D106.C2: now also D105.A2
- net at D23.A1: now also D24.C1
- net at D23.A2: now also D24.C2
- net at D23.A3: now also D24.C3
- net at D16.A1: now also R12.1
- net at D16.A2: now also R13.1
- net at D32.A1: now also R25.1
- net at D32.A2: now also R26.1
- net at D32.A3: now also D33.C3
- net at D144.A1: now also R118.1
- net at D144.A2: now also R119.1
- net at D144.A3: now also R120.1
- net at D144.C1: now also D143.A1
- net at D144.C2: now also D143.A2
- net at D144.C3: now also D143.A3
- net at D139.A1: now also D140.C1
- net at D139.A2: now also D140.C2
- net at D139.A3: now also D140.C3
- net at D139.C1: now also D138.A1
- net at D139.C2: now also D138.A2
- net at D123.A3: now also R101.1
- net at D45.A1: now also D46.C1
- net at D45.A2: now also D46.C2
- net at D45.A3: now also R37.1
- net at D45.C3: now also D44.A3
- net at D76.A1: now also R62.1
- net at D76.A2: now also R63.1
- net at D76.C1: now also D75.A1
- net at D76.C2: now also D75.A2
- net at D61.A1: now also D62.C1
- net at D61.A2: now also D62.C2
- net at D61.A3: now also D62.C3
- net at D141.A3: now also R117.1
- net at D141.C3: now also D140.A3
- net at D95.A1: now also D96.C1
- net at D95.A2: now also D96.C2
- net at D95.A3: now also D96.C3
- net at D95.C1: now also D94.A1
- net at D95.C2: now also D94.A2
- net at D95.C3: now also D94.A3
- net at D129.A1: now also D130.C1
- net at D129.A2: now also D130.C2
- net at D129.A3: now also R107.1
- net at D129.C3: now also D128.A3
- net at D100.A1: now also R82.1
- net at D100.A2: now also R83.1
- net at D100.A3: now also D101.C3
- net at D100.C1: now also D99.A1
- net at D100.C2: now also D99.A2
- net at D20.A1: now also R15.1
- net at D20.A2: now also R16.1
- net at D130.A1: now also D131.C1
- net at D130.A2: now also D131.C2
- net at D130.A3: now also D131.C3
- net at D90.A3: now also R74.1
- net at D90.C1: now also D89.A1
- net at D90.C2: now also D89.A2
- net at D90.C3: now also D89.A3
- net at D105.A3: now also R87.1
- net at D105.C3: now also D104.A3
- net at D34.C1: now also D33.A1
- net at D34.C2: now also D33.A2
- net at D96.A1: now also R78.1
- net at D96.A2: now also R79.1
- net at D96.A3: now also R80.1
- net at D30.A3: now also R24.1
- net at D103.A1: now also D104.C1
- net at D103.A2: now also D104.C2
- net at D103.A3: now also D104.C3
- net at D103.C1: now also D102.A1
- net at D103.C2: now also D102.A2
- net at D104.A1: now also R85.1
- net at D104.A2: now also R86.1
- net at D116.A1: now also R95.1
- net at D116.A2: now also R96.1
- net at D116.C1: now also D115.A1
- net at D116.C2: now also D115.A2
- net at D116.C3: now also D115.A3
- net at D33.A3: now also R27.1
- net at D57.A1: now also D58.C1
- net at D57.A2: now also D58.C2
- net at D57.A3: now also R47.1
- net at D57.C3: now also D56.A3
- net at D140.A1: now also R115.1
- net at D140.A2: now also R116.1
- net at D92.A1: now also R75.1
- net at D92.A2: now also R76.1
- net at D92.A3: now also D93.C3
- net at D128.A1: now also R105.1
- net at D128.A2: now also R106.1
- net at D128.C1: now also D127.A1
- net at D128.C2: now also D127.A2
- net at D128.C3: now also D127.A3
- net at D71.A1: now also D72.C1
- net at D71.A2: now also D72.C2
- net at D71.A3: now also D72.C3
- net at D71.C1: now also D70.A1
- net at D71.C2: now also D70.A2
- net at D71.C3: now also D70.A3
- net at D111.A3: now also R91.1
- net at D24.A1: now also R18.1
- net at D24.A2: now also R19.1
- net at D24.A3: now also R20.1
- net at D98.A1: now also D99.C1
- net at D98.A2: now also D99.C2
- net at D98.A3: now also D99.C3
- net at D135.A3: now also R111.1
- net at D135.C1: now also D134.A1
- net at D135.C2: now also D134.A2
- net at D135.C3: now also D134.A3
- net at D43.A1: now also D44.C1
- net at D43.A2: now also D44.C2
- net at D43.A3: now also D44.C3
- net at D88.A1: now also R72.1
- net at D88.A2: now also R73.1
- net at D88.A3: now also D89.C3
- net at D40.A1: now also R32.1
- net at D40.A2: now also R33.1
- net at D63.A1: now also D64.C1
- net at D63.A2: now also D64.C2
- net at D63.A3: now also R51.1
- net at D63.C1: now also D62.A1
- net at D63.C2: now also D62.A2
- net at D63.C3: now also D62.A3
- net at D101.A1: now also D102.C1
- net at D101.A2: now also D102.C2
- net at D101.A3: now also D102.C3
- net at D81.A3: now also R67.1
- net at D81.C3: now also D80.A3
- net at D72.A1: now also R58.1
- net at D72.A2: now also R59.1
- net at D72.A3: now also R60.1
- net at D36.A1: now also R28.1
- net at D36.A2: now also R29.1
- net at D36.A3: now also R30.1
- net at D64.A1: now also R52.1
- net at D64.A2: now also R53.1
- net at D115.C1: now also D114.A1
- net at D115.C2: now also D114.A2
- net at D132.A1: now also R108.1
- net at D132.A2: now also R109.1
- net at D132.A3: now also R110.1
- net at D132.C1: now also D131.A1
- net at D132.C2: now also D131.A2
- net at D132.C3: now also D131.A3
- net at D99.A3: now also R81.1
- net at D74.A1: now also D75.C1
- net at D74.A2: now also D75.C2
- net at D74.A3: now also D75.C3
- net at D74.C1: now also D73.A1
- net at D74.C2: now also D73.A2
- net at D74.C3: now also D73.A3
- net at D55.A1: now also D56.C1
- net at D55.A2: now also D56.C2
- net at D55.A3: now also D56.C3
- net at D55.C1: now also D54.A1
- net at D55.C2: now also D54.A2
- net at D59.C1: now also D58.A1
- net at D59.C2: now also D58.A2
- net at D59.C3: now also D58.A3
- net at D54.A3: now also R44.1
- net at D93.A1: now also D94.C1
- net at D93.A2: now also D94.C2
- net at D93.A3: now also R77.1
- net at D44.A1: now also R35.1
- net at D44.A2: now also R36.1
- net at D85.A1: now also D86.C1
- net at D85.A2: now also D86.C2
- net at D85.A3: now also D86.C3
- net at D56.A1: now also R45.1
- net at D56.A2: now also R46.1
- net at D113.A1: now also D114.C1
- net at D113.A2: now also D114.C2
- net at D113.A3: now also D114.C3
- net at D80.A1: now also R65.1
- net at D80.A2: now also R66.1
- net at D48.A1: now also R38.1
- net at D48.A2: now also R39.1
- net at D48.A3: now also R40.1
- net at D102.A3: now also R84.1
- net at D84.A1: now also R68.1
- net at D84.A2: now also R69.1
- net at D84.A3: now also R70.1
- net at D75.A3: now also R61.1
- net at D114.A3: now also R94.1
- net at D138.A3: now also R114.1
- new net: D8.A1, R4.1
Other:
- moved on the sheet: D1, D10, D11, D12, D2, D3, D4, D5, D6, D7, D8, D9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

Commit message: cv28 v1.3
Parts:
- R1: renamed from R10; footprint Resistor_THT:R_Axial_DIN0617_L17.0mm_D6.0mm_P20.32mm_Horizontal -> Resistor_THT:R_Axial_DIN0207_L6.3mm_D2.5mm_P10.16mm_Horizontal
- R10: renamed from R3; footprint Resistor_THT:R_Axial_DIN0617_L17.0mm_D6.0mm_P20.32mm_Horizontal -> Resistor_THT:R_Axial_DIN0207_L6.3mm_D2.5mm_P10.16mm_Horizontal
- R100, R101, R102, R103, R104, R105, R106, R107, R108, R109, R11, R110, R111, R112, R113, R114, R115, R116, R117, R118, R119, R12, R120, R13, R14, R15, R16, R17, R18, R19, R20, R21, R22, R23, R24, R25, R26, R27, R28, R29, R30, R31, R32, R33, R34, R35, R36, R37, R38, R39, R40, R41, R42, R43, R44, R45, R46, R47, R48, R49, R50, R51, R52, R53, R54, R55, R56, R57, R58, R59, R60, R61, R62, R63, R64, R65, R66, R67, R68, R69, R70, R71, R72, R73, R74, R75, R76, R77, R78, R79, R80, R81, R82, R83, R84, R85, R86, R87, R88, R89, R90, R91, R92, R93, R94, R95, R96, R97, R98, R99: footprint Resistor_THT:R_Axial_DIN0617_L17.0mm_D6.0mm_P20.32mm_Horizontal -> Resistor_THT:R_Axial_DIN0207_L6.3mm_D2.5mm_P10.16mm_Horizontal
- R2: renamed from R7; footprint Resistor_THT:R_Axial_DIN0617_L17.0mm_D6.0mm_P20.32mm_Horizontal -> Resistor_THT:R_Axial_DIN0207_L6.3mm_D2.5mm_P10.16mm_Horizontal
- R3: renamed from R8; footprint Resistor_THT:R_Axial_DIN0617_L17.0mm_D6.0mm_P20.32mm_Horizontal -> Resistor_THT:R_Axial_DIN0207_L6.3mm_D2.5mm_P10.16mm_Horizontal
- R4: renamed from R9; footprint Resistor_THT:R_Axial_DIN0617_L17.0mm_D6.0mm_P20.32mm_Horizontal -> Resistor_THT:R_Axial_DIN0207_L6.3mm_D2.5mm_P10.16mm_Horizontal
- R5: renamed from R4; footprint Resistor_THT:R_Axial_DIN0617_L17.0mm_D6.0mm_P20.32mm_Horizontal -> Resistor_THT:R_Axial_DIN0207_L6.3mm_D2.5mm_P10.16mm_Horizontal
- R6: renamed from R5; footprint Resistor_THT:R_Axial_DIN0617_L17.0mm_D6.0mm_P20.32mm_Horizontal -> Resistor_THT:R_Axial_DIN0207_L6.3mm_D2.5mm_P10.16mm_Horizontal
- R7: renamed from R6; footprint Resistor_THT:R_Axial_DIN0617_L17.0mm_D6.0mm_P20.32mm_Horizontal -> Resistor_THT:R_Axial_DIN0207_L6.3mm_D2.5mm_P10.16mm_Horizontal
- R8: renamed from R1; footprint Resistor_THT:R_Axial_DIN0617_L17.0mm_D6.0mm_P20.32mm_Horizontal -> Resistor_THT:R_Axial_DIN0207_L6.3mm_D2.5mm_P10.16mm_Horizontal
- R9: renamed from R2; footprint Resistor_THT:R_Axial_DIN0617_L17.0mm_D6.0mm_P20.32mm_Horizontal -> Resistor_THT:R_Axial_DIN0207_L6.3mm_D2.5mm_P10.16mm_Horizontal
